Commit message: proper gazebo params

File: aubo_description/urdf/aubo_i5_gazebo.xacro (robot description, xacro)
@@ -1,27 +1,34 @@
 <?xml version="1.0"?>
 <robot xmlns:xacro="http://www.ros.org/wiki/xacro">
-     <xacro:macro name="aubo_i5_gazebo" params="prefix">
-          <!-- Configure self collision properties per link -->
-          <gazebo reference="${prefix}shoulder_link">
-               <selfCollide>true</selfCollide>
-          </gazebo>
-          <gazebo reference="${prefix}upper_arm_link">
-               <selfCollide>true</selfCollide>
-          </gazebo>
-          <gazebo reference="${prefix}forearm_link">
-               <selfCollide>true</selfCollide>
-          </gazebo>
-          <gazebo reference="${prefix}wrist_1_link">
-               <selfCollide>true</selfCollide>
-          </gazebo>
-          <gazebo reference="${prefix}wrist_3_link">
-               <selfCollide>true</selfCollide>
-          </gazebo>
-          <gazebo reference="${prefix}wrist_2_link">
-               <selfCollide>true</selfCollide>
-          </gazebo>
-          <gazebo reference="${prefix}ee_link">
-               <selfCollide>true</selfCollide>
-          </gazebo>
-     </xacro:macro>
+  <xacro:macro name="aubo_i5_gazebo" params="prefix">
+    <xacro:macro name="aubo_i5_gazebo_link_properties" params="reference">
+      <gazebo reference="${reference}">
+        <kp>1000000.0</kp>
+        <kd>1.0</kd>
+        <mu1>0.8</mu1>
+        <mu2>0.8</mu2>
+        <maxVel>0.0</maxVel>
+        <minDepth>0.001</minDepth>
+        <selfCollide>true</selfCollide>
+      </gazebo>
+    </xacro:macro>
+    <xacro:aubo_i5_gazebo_link_properties reference="${prefix}aubo_i5_base_link" />
+    <xacro:aubo_i5_gazebo_link_properties reference="${prefix}shoulder_link" />
+    <xacro:aubo_i5_gazebo_link_properties reference="${prefix}upper_arm_link" />
+    <xacro:aubo_i5_gazebo_link_properties reference="${prefix}forearm_link" />
+    <xacro:aubo_i5_gazebo_link_properties reference="${prefix}wrist_1_link" />
+    <xacro:aubo_i5_gazebo_link_properties reference="${prefix}wrist_2_link" />
+    <xacro:aubo_i5_gazebo_link_properties reference="${prefix}wrist_3_link" />
+    <xacro:macro name="aubo_i5_gazebo_joint_properties" params="reference">
+      <gazebo reference="${reference}">
+        <implicitSpringDamper>true</implicitSpringDamper>
+      </gazebo>
+    </xacro:macro>
+    <xacro:aubo_i5_gazebo_link_properties reference="${prefix}shoulder_pan_joint" />
+    <xacro:aubo_i5_gazebo_link_properties reference="${prefix}shoulder_lift_joint" />
+    <xacro:aubo_i5_gazebo_link_properties reference="${prefix}elbow_joint" />
+    <xacro:aubo_i5_gazebo_link_properties reference="${prefix}wrist_1_joint" />
+    <xacro:aubo_i5_gazebo_link_properties reference="${prefix}wrist_2_joint" />
+    <xacro:aubo_i5_gazebo_link_properties reference="${prefix}wrist_3_joint" />
+  </xacro:macro>
 </robot>
