Commit message: moveit config aubo i5

File: aubo_description/urdf/aubo_i5.xacro (robot description, xacro)
@@ -9,8 +9,14 @@
     prefix=""
     parent="world"
-    hw_interface="hardware_interface/EffortJointInterface"
+    hw_interface="hardware_interface/PositionJointInterface"
   >
     <origin xyz="0.0 0.0 0.0" rpy="0.0 0.0 0.0" />
   </xacro:aubo_i5>
+  <link name="teleop_link" />
+  <joint name="teleop_link_joint" type="fixed">
+    <parent link="ee_link" />
+    <child link="teleop_link" />
+    <origin rpy="${-pi/2} 0 ${-pi/2}" xyz="0 0 0" />
+  </joint>
   <gazebo>
     <plugin name="ros_control" filename="libgazebo_ros_control.so"></plugin>

File: aubo_description/urdf/aubo_i5_macro.xacro (robot description, xacro)
@@ -14,5 +14,5 @@
     <xacro:property name="max_effort_1" value="150.0" />
     <xacro:property name="max_effort_2" value="28.0" />
-    <xacro:property name="max_velocity" value="${pi}" />
+    <xacro:property name="max_velocity" value="${1}" />
     <!-- INERTIA -->
     <xacro:macro name="I5_BaseLink_Inertia">
