Commit message: add ee_link

File: aubo_description/urdf/aubo_i5_macro.xacro (robot description, xacro)
@@ -273,4 +273,17 @@
       <limit lower="-3.04" upper="3.04" effort="300" velocity="100" />
     </joint>
+    <link name="${prefix}ee_link">
+      <collision>
+        <geometry>
+          <box size="0.01 0.01 0.01" />
+        </geometry>
+        <origin rpy="0 0 0" xyz="-0.01 0 0" />
+      </collision>
+    </link>
+    <joint name="${prefix}ee_fixed_joint" type="fixed">
+      <parent link="${prefix}wrist_3_link" />
+      <child link="${prefix}ee_link" />
+      <origin rpy="${pi} ${-pi/2} ${pi/2}" xyz="0.0 0.0 0.0" />
+    </joint>
     <joint name="${prefix}aubo_i5_base_joint" type="fixed">
       <parent link="${parent}"/>

Commit message: fix aubo_msgs dependency bug

File: aubo_description/urdf/aubo_i5_macro.xacro (robot description, xacro)
@@ -238,5 +238,5 @@
       <limit lower="-3.04" upper="3.04" effort="300" velocity="100" />
     </joint>
-    <joint name="${prefix}should_lift_joint" type="revolute">
+    <joint name="${prefix}shoulder_lift_joint" type="revolute">
       <origin xyz="0 0.1215 0" rpy="-1.5708 -1.5708 0" />
       <parent link="${prefix}shoulder_link" />

Commit message: fix mass and inertia, remove unnecessary packages

File: aubo_description/urdf/aubo_i5_macro.xacro (robot description, xacro)
@@ -3,5 +3,6 @@
   <xacro:include filename="$(find aubo_description)/urdf/aubo_i5_transmission.xacro" />
   <xacro:include filename="$(find aubo_description)/urdf/aubo_i5_gazebo.xacro" />
-  <xacro:macro name="aubo_i5" params="
+  <xacro:macro name="aubo_i5"
+    params="
   prefix
   parent
@@ -13,79 +14,41 @@
     <!-- INERTIA -->
     <xacro:macro name="I5_BaseLink_Inertia">
-      <origin xyz="-1.4795E-13 0.0015384 0.020951" rpy="0 0 0" />
+      <origin xyz="1.1888811586008421e-07 0.0015716172771383882 0.020944607206477398" rpy="0 0 0" />
       <mass value="0.83419" />
-      <inertia
-        ixx="0.0014414"
-        ixy="7.8809E-15"
-        ixz="8.5328E-16"
-        iyy="0.0013542"
-        iyz="-1.4364E-05"
-        izz="0.0024659" />
+      <inertia ixx="${0.011226*0.12799542569}" iyy="${0.010532*0.12799542569}"
+        izz="${0.019183*0.12799542569}" ixy="-0.0" iyz="${-0.000114*0.12799542569}" ixz="-0.0" />
     </xacro:macro>
     <xacro:macro name="I5_Shoulder_Inertia">
-      <origin xyz="0.0 0.006 -0.002"
-        rpy="0 0 0" />
+      <origin xyz="0.0 0.006 -0.002" rpy="0 0 0" />
       <mass value="5.05" />
-      <inertia ixx="0.0148"
-        ixy="0"
-        ixz="0"
-        iyy="0.0143"
-        iyz="-0.0"
-        izz="0.0095" />
+      <inertia ixx="0.0148" ixy="0" ixz="0" iyy="0.0143" iyz="-0.0" izz="0.0095" />
     </xacro:macro>
     <xacro:macro name="I5_UpperArm_Inertia">
-      <origin xyz="0.304 0.0 -0.03"
-        rpy="0 0 0" />
+      <origin xyz="0.20400000738607602 0.0003079721588177273 0.020108705518388777" rpy="0 0 0" />
       <mass value="11.90" />
-      <inertia ixx="0.0305"
-        ixy="0"
-        ixz="0"
-        iyy="0.4505"
-        iyz="0"
-        izz="0.0095" />
+      <inertia ixx="${0.133789*0.21958145116}" iyy="${1.548798*0.21958145116}"
+        izz="${1.5133*0.21958145116}" ixy="${-0.0*0.21958145116}" iyz="${2.3e-05*0.21958145116}"
+        ixz="${0.0*0.21958145116}" />
     </xacro:macro>
     <xacro:macro name="I5_ForeArm_Inertia">
-      <origin xyz="0.415 0.0 0.0992"
-        rpy="0 0 0" />
+      <origin xyz="0.18880713458962045 8.0702133231828e-06 0.09802927852704038" rpy="0 0 0" />
       <mass value="3.3" />
-      <inertia ixx="0.0033"
-        ixy="0"
-        ixz="0.0009"
-        iyy="0.0575"
-        iyz="0"
-        izz="0.0565" />
+      <inertia ixx="${0.016448*0.18731379107}" iyy="${0.345066*0.18731379107}" izz="${0.343039*0.18731379107}" ixy="${1.3e-05*0.18731379107}" iyz="${2e-06*0.18731379107}"
+        ixz="${-0.005687*0.18731379107}" />
     </xacro:macro>
     <xacro:macro name="I5_Wrist1_Inertia">
-      <origin xyz="0.0 0.0028 -0.003"
-        rpy="0 0 0" />
+      <origin xyz="0.0 0.0028 -0.003" rpy="0 0 0" />
       <mass value="1.62" />
-      <inertia ixx="0.0023"
-        ixy="0"
-        ixz="0"
-        iyy="0.0013"
-        iyz="0.0"
-        izz="0.0022" />
+      <inertia ixx="0.0023" ixy="0" ixz="0" iyy="0.0013" iyz="0.0" izz="0.0022" />
     </xacro:macro>
     <xacro:macro name="I5_Wrist2_Inertia">
-      <origin xyz="0.0 -0.0028 -0.003"
-        rpy="0 0 0" />
+      <origin xyz="0.0 -0.0028 -0.003" rpy="0 0 0" />
       <mass value="1.62" />
-      <inertia ixx="0.0023"
-        ixy="0"
-        ixz="0"
-        iyy="0.0013"
-        iyz="0.0"
-        izz="0.0022" />
+      <inertia ixx="0.0023" ixy="0" ixz="0" iyy="0.0013" iyz="0.0" izz="0.0022" />
     </xacro:macro>
     <xacro:macro name="I5_Wrist3_Inertia">
-      <origin xyz="0.0 0.0 -0.0071"
-        rpy="0 0 0" />
-      <mass value="0.40" />
-      <inertia ixx="0.013939"
-        ixy="0"
-        ixz="0"
-        iyy="0.013988"
-        iyz="0.0"
-        izz="0.0224092" />
+        <origin xyz="3.8199537218366924e-05 -6.891283689656669e-05 -0.021357543727161605" rpy="0 0 0"/>
+        <mass value="${1.2143524682183242*0.32939365667}"/>
+        <inertia ixx="${0.000545*0.32939365667}" iyy="${0.000549*0.32939365667}" izz="${0.000814*0.32939365667}" ixy="${-0.0*0.32939365667}" iyz="${0.0*0.32939365667}" ixz="${-0.0*0.32939365667}"/>
     </xacro:macro>
     <!-- LINKS -->
@@ -236,5 +199,5 @@
       <child link="${prefix}shoulder_link" />
       <axis xyz="0 0 1" />
-      <limit lower="-3.04" upper="3.04" effort="300" velocity="100" />
+      <limit lower="-3.04" upper="3.04" effort="150" velocity="${pi}" />
     </joint>
     <joint name="${prefix}shoulder_lift_joint" type="revolute">
@@ -243,5 +206,5 @@
       <child link="${prefix}upper_arm_link" />
       <axis xyz="0 0 1" />
-      <limit lower="-3.04" upper="3.04" effort="300" velocity="100" />
+      <limit lower="-3.04" upper="3.04" effort="150" velocity="${pi}" />
     </joint>
     <joint name="${prefix}elbow_joint" type="revolute">
@@ -250,5 +213,5 @@
       <child link="${prefix}forearm_link" />
       <axis xyz="0 0 1" />
-      <limit lower="-3.04" upper="3.04" effort="300" velocity="100" />
+      <limit lower="-3.04" upper="3.04" effort="150" velocity="${pi}" />
     </joint>
     <joint name="${prefix}wrist_1_joint" type="revolute">
@@ -257,5 +220,5 @@
       <child link="${prefix}wrist_1_link" />
       <axis xyz="0 0 1" />
-      <limit lower="-3.04" upper="3.04" effort="300" velocity="100" />
+      <limit lower="-3.04" upper="3.04" effort="28" velocity="${pi}" />
     </joint>
     <joint name="${prefix}wrist_2_joint" type="revolute">
@@ -264,5 +227,5 @@
       <child link="${prefix}wrist_2_link" />
       <axis xyz="0 0 1" />
-      <limit lower="-3.04" upper="3.04" effort="300" velocity="100" />
+      <limit lower="-3.04" upper="3.04" effort="28" velocity="${pi}" />
     </joint>
     <joint name="${prefix}wrist_3_joint" type="revolute">
@@ -271,5 +234,5 @@
       <child link="${prefix}wrist_3_link" />
       <axis xyz="0 0 1" />
-      <limit lower="-3.04" upper="3.04" effort="300" velocity="100" />
+      <limit lower="-3.04" upper="3.04" effort="28" velocity="${pi}" />
     </joint>
     <link name="${prefix}ee_link">
@@ -287,7 +250,7 @@
     </joint>
     <joint name="${prefix}aubo_i5_base_joint" type="fixed">
-      <parent link="${parent}"/>
-      <child link="${prefix}aubo_i5_base_link"/>
-      <xacro:insert_block name="origin"/>
+      <parent link="${parent}" />
+      <child link="${prefix}aubo_i5_base_link" />
+      <xacro:insert_block name="origin" />
     </joint>
   </xacro:macro>

Commit message: update aubo_i5_macro.xacro

File: aubo_description/urdf/aubo_i5_macro.xacro (robot description, xacro)
@@ -12,4 +12,7 @@
     <xacro:aubo_i5_transmission prefix="${prefix}" hw_interface="${hw_interface}" />
     <xacro:aubo_i5_gazebo prefix="${prefix}" />
+    <xacro:property name="max_effort_1" value="150.0" />
+    <xacro:property name="max_effort_2" value="28.0" />
+    <xacro:property name="max_velocity" value="${pi}" />
     <!-- INERTIA -->
     <xacro:macro name="I5_BaseLink_Inertia">
@@ -199,5 +202,5 @@
       <child link="${prefix}shoulder_link" />
       <axis xyz="0 0 1" />
-      <limit lower="-3.04" upper="3.04" effort="150" velocity="${pi}" />
+      <limit lower="-3.04" upper="3.04" effort="${max_effort_1}" velocity="${max_velocity}" />
     </joint>
     <joint name="${prefix}shoulder_lift_joint" type="revolute">
@@ -206,5 +209,5 @@
       <child link="${prefix}upper_arm_link" />
       <axis xyz="0 0 1" />
-      <limit lower="-3.04" upper="3.04" effort="150" velocity="${pi}" />
+      <limit lower="-3.04" upper="3.04" effort="${max_effort_1}" velocity="${max_velocity}" />
     </joint>
     <joint name="${prefix}elbow_joint" type="revolute">
@@ -213,5 +216,5 @@
       <child link="${prefix}forearm_link" />
       <axis xyz="0 0 1" />
-      <limit lower="-3.04" upper="3.04" effort="150" velocity="${pi}" />
+      <limit lower="-3.04" upper="3.04" effort="${max_effort_1}" velocity="${max_velocity}" />
     </joint>
     <joint name="${prefix}wrist_1_joint" type="revolute">
@@ -220,5 +223,5 @@
       <child link="${prefix}wrist_1_link" />
       <axis xyz="0 0 1" />
-      <limit lower="-3.04" upper="3.04" effort="28" velocity="${pi}" />
+      <limit lower="-3.04" upper="3.04" effort="${max_effort_2}" velocity="${max_velocity}" />
     </joint>
     <joint name="${prefix}wrist_2_joint" type="revolute">
@@ -227,5 +230,5 @@
       <child link="${prefix}wrist_2_link" />
       <axis xyz="0 0 1" />
-      <limit lower="-3.04" upper="3.04" effort="28" velocity="${pi}" />
+      <limit lower="-3.04" upper="3.04" effort="${max_effort_2}" velocity="${max_velocity}" />
     </joint>
     <joint name="${prefix}wrist_3_joint" type="revolute">
@@ -234,5 +237,5 @@
       <child link="${prefix}wrist_3_link" />
       <axis xyz="0 0 1" />
-      <limit lower="-3.04" upper="3.04" effort="28" velocity="${pi}" />
+      <limit lower="-3.04" upper="3.04" effort="${max_effort_2}" velocity="${max_velocity}" />
     </joint>
     <link name="${prefix}ee_link">

Commit message: updated effort vel limits

File: aubo_description/urdf/aubo_i5_macro.xacro (robot description, xacro)
@@ -12,7 +12,7 @@
     <xacro:aubo_i5_transmission prefix="${prefix}" hw_interface="${hw_interface}" />
     <xacro:aubo_i5_gazebo prefix="${prefix}" />
-    <xacro:property name="max_effort_1" value="150.0" />
-    <xacro:property name="max_effort_2" value="28.0" />
-    <xacro:property name="max_velocity" value="${1}" />
+    <xacro:property name="max_effort_1" value="300.0" />
+    <xacro:property name="max_effort_2" value="50.0" />
+    <xacro:property name="max_velocity" value="${pi}" />
     <!-- INERTIA -->
     <xacro:macro name="I5_BaseLink_Inertia">
